Commit message: initial commmit

File: src/my_robot/urdf/my_robot.xacro (robot description, xacro)
@@ -154,9 +154,19 @@
 		<axis xyz="0 1 0" rpy="0 0 0"/>
 	</joint>
-<!-- Lidar sensor -->
-  <link name='hokuyo'>
-    <inertial>
-      <mass value="1e-5"/>
-      <origin xyz="0.0 0 0" rpy=" 0 0 0"/>
+<!-- Camera link optical -->
+<!-- >	<link name="camera_link_optical">
+	</link>
+	<joint name="camera_optical_joint" type="fixed">
+		<origin xyz="0 0 0" rpy="-1.5707 0 -1.5707"/>
+		<parent link="camera_link"/>
+		<child link="camera_link_optical"/>
+	</joint>
+-->
+  <link name="camera_link_optical">
+    <pose>0 0 0 0 0 0</pose>
+    <inertial>
+      <mass value="0.1"/>
+      <origin xyz="0.0 0 0" rpy=" 0 0 0"/>
+      <box_inertia m="0.1" x="0.05" y="0.05" z="0.05"/>
       <inertia
           ixx="1e-6" ixy="0" ixz="0"
@@ -165,4 +175,34 @@
       />
     </inertial>
+    <collision name='collision'>
+      <origin xyz="0 0 0" rpy=" 0 0 0"/>
+      <geometry>
+        <box size=".05 .05 .05"/>
+      </geometry>
+    </collision>
+    <visual name='camera_optical_visual'>
+      <origin xyz="0 0 0" rpy=" 0 0 0"/>
+      <geometry>
+        <box size=".05 .05 .05"/>
+      </geometry>
+    </visual>
+  </link>
+  <joint name="camera_optical_joint" type="fixed">
+    <origin xyz="0.2 0 0" rpy="-1.5707 0 -1.5707"/>
+    <parent link="chassis"/>
+    <child link="camera_link_optical"/>
+    <axis xyz="0.0 1.0 0.0"/>
+  </joint>
+<!-- Lidar sensor -->
+  <link name='hokuyo'>
+    <inertial>
+      <mass value="1e-5"/>
+      <origin xyz="0.0 0 0" rpy=" 0 0 0"/>
+      <inertia
+          ixx="1e-6" ixy="0" ixz="0"
+          iyy="1e-6" iyz="0"
+          izz="1e-6"
+      />
+    </inertial>
     <collision name='hokuyo_collision'>
       <origin xyz="0 0 0" rpy=" 0 0 0"/>
